Commit message: version update in rosinstall file

File: configuration_files/hokuyo3d.urdf (robot description, URDF)
Before this commit: robot hokuyo3d, 4 links, 3 joints
Joints:
- joint base_to_laser: origin xyz=0.071 0.0 0.0055 rpy=0.0 0.0 0.0 -> xyz=0.071 0.0 0.055 rpy=0.0 0.0 0.0

File: configuration_files/hokuyo3d_gx5.urdf (robot description, URDF)
Before this commit: robot hokuyo3d, 4 links, 3 joints
Joints:
- joint base_to_imu: origin xyz=0.01 0.0 0.0056 rpy=0.0 0.0 1.571 -> xyz=0.02 0.0 0.1 rpy=0.0 0.0 -1.571
- joint base_to_laser: origin xyz=0.071 0.0 0.0055 rpy=0.0 0.0 0.0 -> xyz=0.071 0.0 0.055 rpy=0.0 0.0 0.0
- joint base_to_mag: origin xyz=0.01 0.0 0.0 rpy=-1.571 -1.571 1.571 -> xyz=0.02 0.0 0.1 rpy=-1.571 -1.571 1.571
