Commit message: add some modifies

File: configuration_files/hokuyo3d_gx5.urdf (robot description, URDF)
Before this commit: robot hokuyo3d, 4 links, 3 joints
Links:
- removed link hokuyo3d_link
- removed link hokuyo3d_mag
- added link base_link
Joints:
- removed joint base_to_mag
- joint base_to_imu: origin xyz=0.02 0.0 0.1 rpy=0.0 0.0 -1.571 -> xyz=0.02 0.0 0.1 rpy=0.0 3.142 -1.571; parent hokuyo3d_link -> base_link
- joint base_to_laser: parent hokuyo3d_link -> base_link

Commit message: add files for docker

File: configuration_files/hokuyo3d_gx5.urdf (robot description, URDF)
Before this commit: robot hokuyo3d, 3 links, 2 joints
Links:
- added link hokuyo3d_mag
Joints:
- added joint base_to_mag: type fixed, parent base_link, child hokuyo3d_mag, origin xyz=0.02 0.0 0.1 rpy=-1.571 -1.571 1.571

Commit message: modified bugs to work on 2d and 3d

File: configuration_files/hokuyo3d_gx5.urdf (robot description, URDF)
Before this commit: robot hokuyo3d, 4 links, 3 joints
Joints:
- joint base_to_imu: origin xyz=0.02 0.0 0.1 rpy=0.0 3.142 -1.571 -> xyz=0.02 0.0 0.1 rpy=0.0 0.0 -1.571
